File: src/CreativePad.kicad_pcb (KiCad board)
At the start: 2 copper layers, 66 parts, among them SW2 TS342A2P-WZ, U1 TPMIC5219-2.8YM5, U17 RP2040_C2961140, U19 W25Q128JWPIQ, U2 AMS1117-3.3, X2 DSX321G-12MHZ

Commit message: Day 5 - P1
Parts:
- S1, S10, S11, S12, S13, S14, S15, S16, S2, S3, S4, S5, S6, S7, S8, S9: moved to B.Cu
- moved D1 119.8 mm to (31.2, 83.7)
- moved D5 118.6 mm to (31.2, 102.8)
- moved D9 117.5 mm to (31.2, 121.8)
- moved D13 116.7 mm to (31.2, 140.9)
- moved VR2 114.5 mm to (90.6, 52.6)
- moved S16 109.0 mm to (34.1, 135.2), turned to 180 degrees
- moved VR1 104.4 mm to (105.8, 36.4)
- moved D2 102.7 mm to (50.2, 83.7)
- moved S12 102.6 mm to (34.1, 116.1), turned to 180 degrees
- moved D6 101.1 mm to (50.2, 102.8)
- moved D10 99.8 mm to (50.2, 121.8)
- moved D14 98.6 mm to (50.2, 140.9)
- moved C11 88.4 mm to (130.3, 49.8)
- moved C12 88.4 mm to (172.6, 53.7)
- moved C13 88.4 mm to (130.3, 52.5)
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
Commit message: Day 5
Parts:
- removed the D3 at (69.3, 83.7)
- removed REF**: OLED-SMD_HS20HS072RX, easyeda2kicad:OLED-SMD_HS20HS072RX
- added D3 (x2): Diode, ScottoKeebs_Components:Diode_DO-35, F.Cu at (69.3, 83.7)
- S1, S10, S11, S12, S13, S14, S15, S16, S2, S3, S4, S5, S6, S7, S8, S9: footprint ScottoKeebs_Scotto:MX_Hotswap_1.00u -> Switch_Keyboard_Hotswap_Kailh:SW_Hotswap_Kailh_MX_1.00u; moved to F.Cu
- moved C15 89.2 mm to (84.3, 44.0)
- moved R2 82.4 mm to (83.8, 45.6)
- moved SW2 79.7 mm to (90.6, 29.7)
- moved U1 77.2 mm to (96.5, 39.9)
- moved C12 76.5 mm to (97.0, 42.4)
- moved U17 71.2 mm to (81.7, 58.9)
- moved R3 71.0 mm to (95.4, 65.1)
- moved X2 70.2 mm to (97.4, 52.8)
- moved R8 67.6 mm to (98.5, 65.1)
- moved U19 64.6 mm to (97.0, 59.9)
- moved USB2 63.4 mm to (80.8, 31.5), turned to 180 degrees
- moved U2 62.8 mm to (90.6, 45.6)
- moved R6 58.8 mm to (89.0, 40.9)
- moved S1 57.1 mm to (34.1, 78.0), turned to 0 degrees
- moved S4 57.1 mm to (91.2, 78.0), turned to 0 degrees
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Connections:
- S1 pad 1: ROW0 -> (no net)
- S1 pad 2: Net-(D1-A) -> (no net)
Routing:
- net COL0: track 0.00 -> 59.9 mm
- net Net-(D8-A): track 0.00 -> 57.1 mm
- net Net-(D7-A): track 0.00 -> 57.1 mm
- net Net-(D6-A): track 0.00 -> 57.1 mm
- net Net-(D5-A): track 0.00 -> 57.1 mm

Commit message: Day 6
Parts:
- removed the D3 at (69.3, 83.7) (x2)
- added D3: Diode, ScottoKeebs_Components:Diode_DO-35, F.Cu at (81.1, 76.7)
- U17: value RP2040_C2961140 -> RP2040
- X2: value DSX321G-12MHZ -> 12MHZ
- moved S13 57.9 mm to (33.5, 131.3)
- moved S5 57.9 mm to (33.5, 93.2)
- moved S9 57.9 mm to (33.5, 112.3)
- moved S12 56.6 mm to (90.6, 112.3)
- moved S16 56.6 mm to (90.6, 131.3)
- moved S8 56.6 mm to (90.6, 93.2)
- moved C14 43.6 mm to (100.8, 28.4)
- moved C17 43.3 mm to (100.2, 26.6), turned to 180 degrees
- moved C11 36.4 mm to (97.3, 31.3), turned to 180 degrees
- moved C8 35.7 mm to (101.4, 30.7)
- moved C9 29.0 mm to (99.5, 38.4), turned to -90 degrees
- moved C1 28.8 mm to (78.2, 36.1)
- moved C7 28.2 mm to (97.2, 28.9)
- moved R8 26.0 mm to (76.7, 51.0)
- moved C2 25.3 mm to (83.4, 36.1), turned to 180 degrees
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Connections:
- S1 pad 1: (no net) -> ROW0
- S1 pad 2: (no net) -> Net-(D1-A)
Routing:
- net GND: track 0.00 -> 257.5 mm, vias 0 -> 2
- net +3V3: track 0.00 -> 176.6 mm, vias 0 -> 2
- net COL3: track 0.00 -> 165.0 mm, vias 0 -> 1
- net COL2: track 0.00 -> 153.6 mm
- net ROW0: track 0.00 -> 121.1 mm, vias 0 -> 1
- net COL1: track 0.00 -> 112.1 mm, vias 0 -> 1
- net ROW1: track 0.00 -> 101.9 mm, vias 0 -> 1
- net ROW3: track 0.00 -> 95.2 mm, vias 0 -> 1
- net ROW2: track 0.00 -> 85.5 mm, vias 0 -> 1
- net QSS: track 0.00 -> 70.2 mm, vias 0 -> 4
- net +1V1: track 0.00 -> 69.7 mm, vias 0 -> 2
- net (no net): track 0.00 -> 65.9 mm, vias 0 -> 3
- net +5V: track 0.00 -> 58.6 mm, vias 0 -> 2
- net Net-(D8-A): track 57.1 -> 3.68 mm
- net Net-(D7-A): track 57.1 -> 3.68 mm
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
Commit message: Day 8
Parts:
- removed C11: 100nF, easyeda2kicad:C0603
- removed R3: 1kΩ, easyeda2kicad:R0402
- removed R5, R7: 1.5kΩ, easyeda2kicad:R0603
- removed SW2: TS342A2P-WZ, easyeda2kicad:SW-SMD_L4.0-W2.9-LS5.0
- removed U17: RP2040, easyeda2kicad:QFN-56_L7.0-W7.0-P0.40-TL-EP4.0
- removed U19: W25Q128JWPIQ, easyeda2kicad:WSON-8_L6.0-W5.0-P1.27-BL-EP
- removed USB2: TYPE-C 16PIN 2MD(073), easyeda2kicad:USB-C-SMD_TYPE-C-6PIN-2MD-073
- added C16: 100n, Capacitor_SMD:C_0402_1005Metric, F.Cu at (96.0, 52.2)
- added J1: USBC_2.0_Receptacle_16P, Connector_USB:USB_C_Receptacle_GCT_USB4110, F.Cu at (82.9, 27.8)
- added R12: 1k, Resistor_SMD:R_0402_1005Metric, F.Cu at (92.4, 40.9)
- added R4: 5.1kΩ, easyeda2kicad:R0603, F.Cu at (81.7, 35.1)
- added R9: 5.1kΩ, easyeda2kicad:R0603, F.Cu at (84.7, 35.5)
- added SW1: TS342A2P-WZ, easyeda2kicad:SW-SMD_L4.0-W2.9-LS5.0, F.Cu at (94.2, 28.4)
- added U3: RP2040, RP2040_minimal_r2:RP2040-QFN-56, F.Cu at (82.7, 56.1)
- added U5: W25Q32JVSS, Package_SO:SOIC-8_5.3x5.3mm_P1.27mm, F.Cu at (93.6, 46.8)
- R1: value 5.1kΩ -> DNF; footprint easyeda2kicad:R0603 -> Resistor_SMD:R_0402_1005Metric
- R2: value 1kΩ -> 1.5kΩ; footprint easyeda2kicad:R0402 -> easyeda2kicad:R0603
- R6: value 5.1kΩ -> 1.5kΩ
- X2: value 12MHZ -> DSX321G-12MHZ
- moved C8 43.1 mm to (75.6, 65.3)
- moved C17 41.1 mm to (82.2, 63.5), turned to 0 degrees
- moved C7 40.7 mm to (75.6, 63.5)
- moved C6 40.0 mm to (72.6, 65.3)
- moved C13 39.4 mm to (78.7, 61.7)
- moved C9 34.0 mm to (78.7, 65.3), turned to 0 degrees
- moved C15 32.1 mm to (76.3, 34.3), turned to -90 degrees
- moved C3 28.0 mm to (72.6, 63.5)
- moved C10 24.8 mm to (78.7, 63.5)
- moved C1 24.1 mm to (101.2, 43.2)
- moved R2 21.0 mm to (83.9, 48.6), turned to 0 degrees
- moved R1 20.3 mm to (94.9, 50.4)
- moved C2 18.6 mm to (101.2, 41.5), turned to 0 degrees
- moved C5 18.6 mm to (82.2, 65.3)
- moved R6 14.0 mm to (85.7, 50.4), turned to 0 degrees
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Connections:
- R1 pad 1: Net-(USB2-CC2) -> +3V3
- R1 pad 2: GND -> QSS
- R2 pad 2: QSS -> USB_DP
- R6 pad 2: GND -> USB_DN
Routing:
- net (no net): track 65.9 -> 0.00 mm, vias 3 -> 0
- net QSS: track 70.2 -> 44.5 mm, vias 4 -> 7
- net +3V3: track 176.6 -> 151.3 mm, vias 2 -> 0
- net Net-(U17-USB_DM): track 24.9 -> 0.00 mm, vias 4 -> 0
- net GND: track 257.5 -> 232.6 mm, vias 2 -> 4
- net Net-(U17-USB_DP): track 22.6 -> 0.00 mm, vias 4 -> 0
- net QSD3: track 49.1 -> 27.4 mm
- net +5V: track 58.6 -> 37.1 mm
- net +1V1: track 69.7 -> 50.9 mm, vias 2 -> 3
- net Net-(U3-USB_DM): track 21.2 -> 2.65 mm
- net DSDA: track 28.8 -> 45.0 mm
- net DRST: track 18.8 -> 34.9 mm
- net Net-(R12-Pad2): track 0.00 -> 14.9 mm, vias 0 -> 2
- net USB_DN: track 12.8 -> 25.7 mm, vias 0 -> 2
- net XOUT: track 3.11 -> 12.6 mm
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- added copper zone on B.Cu, net (none)
- added copper zone on F.Cu, net (none)
Other:
- board outline added: 81.6 x 117.5 mm

Commit message: Day 8 - Part 2
Parts:
- J1: footprint Connector_USB:USB_C_Receptacle_GCT_USB4110 -> Connector_USB:USB_C_Receptacle_HCTL_HC-TYPE-C-16P-01A
Routing:
- net GND: track 232.6 -> 229.8 mm
- net USB_DP: track 25.7 -> 27.9 mm
- net +5V: track 37.1 -> 38.6 mm
