File: src/CreativePad.kicad_pcb (KiCad board)
At the start: 2 copper layers, 81.6 x 117.5 mm, 65 parts, among them J1 USBC_2.0_Receptacle_16P, SW1 TS342A2P-WZ, U1 TPMIC5219-2.8YM5, U2 AMS1117-3.3, U3 RP2040, U5 W25Q32JVSS, X2 DSX321G-12MHZ

Commit message: Day 9
Parts:
- added H1: MountingHole, MountingHole:MountingHole_2.2mm_M2, F.Cu at (25.5, 28.2)
- added H2: MountingHole, MountingHole:MountingHole_2.2mm_M2, F.Cu at (100.1, 59.9)
- added H3: MountingHole, MountingHole:MountingHole_2.2mm_M2, F.Cu at (62.0, 121.8)
- added H4: MountingHole, MountingHole:MountingHole_2.2mm_M2, F.Cu at (100.7, 139.3)
Other:
- board text added: "Made By CherryTree56567 @CT5"
